Commit message: Add ZED X perception pipeline with kiwicampus semantic segmentation
New avros_perception package bridges ZED X cameras to Nav2 via
kiwicampus/semantic_segmentation_layer. Single front camera today;
pipeline abstraction (stub / HSV / ONNX) lets us swap CV implementations
without touching Nav2. Verified end-to-end on Jetson Orin: stripe
injection through the stub produces LETHAL cost cells in the local
costmap.

Stack changes:
- avros_perception ament_python package: perception_node with swappable
  Pipeline interface (stub only today), message-filters sync of ZED RGB
  + organized cloud, publishes mask/confidence/cloud/labels with shared
  header.stamp. Auto-resizes image to cloud HxW (they diverge under v5
  wrapper defaults). class_map.yaml is single source of truth for class
  IDs -> LabelInfo.
- zed-ros2-wrapper v5.2.2 in avros.repos. Launched via the wrapper's
  zed_camera.launch.py (wrapper is a metapackage; camera is a
  stereolabs::ZedCamera composable component).
- kiwicampus/semantic_segmentation_layer humble branch + PR #1 carry
  patch (Humble build fix: swap modern imported CMake targets for
  ament_target_dependencies, add <deque>). Applied by
  scripts/apply_kiwicampus_patches.sh after vcs import.
- URDF uses <xacro:include .../zed_macro.urdf.xacro> + <xacro:zed_camera
  name="zed_front" model="zedx"> so the full frame chain the wrapper
  publishes into (camera_link / left_camera_frame_optical / etc) is in
  the TF tree. Hand-rolled single link was insufficient.
- nav2_params*.yaml: local_costmap gets a semantic_front plugin block
  with class_types nested inside the per-source observation block (the
  plugin requires this; top-level class_types fails init).
- navigation.launch.py: enable_perception arg gates the perception node
  include; enable_zed_front plumbs through sensors/localization/nav.

Known gotchas documented in CLAUDE.md Known Issues:
- namespace+node_name collision in wrapper -> pass only camera_name
- v5 topic path is rgb/color/rect/image (not rgb/image_rect_color)
- depth_mode PERFORMANCE / HD720 no longer valid in v5
- serial_number is a launch arg, not YAML param
- image and cloud HxW diverge (perception_node auto-resizes)

Full session log in docs/CHANGELOG_2026-04-24.md.

Co-Authored-By: Claude Opus 4.7 (1M context) <noreply@anthropic.com>

File: src/avros_bringup/urdf/avros.urdf.xacro (robot description, xacro)
@@ -4,4 +4,6 @@
   <xacro:property name="wheelbase" value="1.23"/>
   <xacro:property name="track_width" value="0.9"/>
+  <!-- Optional frames. Pass via xacro args, e.g. xacro avros.urdf.xacro enable_zed_back:=true -->
+  <xacro:arg name="enable_zed_back" default="false"/>
   <!-- ============================================================ -->
   <!-- base_link: center of rear axle at ground level               -->
@@ -98,4 +100,22 @@
   </joint>
   <!-- ============================================================ -->
+  <!-- Camera: ZED X Front (GMSL) — via stock Stereolabs macro      -->
+  <!-- Creates the full frame chain (camera_link, left_camera_frame,-->
+  <!-- right_camera_frame, camera_center, imu_link) that the ZED    -->
+  <!-- wrapper publishes image/cloud frame_ids against. We attach   -->
+  <!-- the camera_link root to base_link via a separate joint.      -->
+  <!-- TODO: Measure exact mount position on real vehicle           -->
+  <!-- ============================================================ -->
+  <xacro:include filename="$(find zed_wrapper)/urdf/zed_macro.urdf.xacro"/>
+  <xacro:zed_camera name="zed_front" model="zedx">
+    <origin xyz="0 0 0" rpy="0 0 0"/>    <!-- gnss_origin block, unused (enable_gnss=false) -->
+  </xacro:zed_camera>
+  <joint name="zed_front_mount_joint" type="fixed">
+    <parent link="base_link"/>
+    <child link="zed_front_camera_link"/>
+    <!-- TODO: Measure on vehicle. Approximate: front center, roof height, facing +X -->
+    <origin xyz="1.0 0.0 0.9" rpy="0 0 0"/>
+  </joint>
+  <!-- ============================================================ -->
   <!-- Camera: ZED X Left (GMSL)                                    -->
   <!-- TODO: Measure exact mount position on real vehicle           -->
@@ -134,20 +154,23 @@
   </joint>
   <!-- ============================================================ -->
-  <!-- Camera: ZED X Back (GMSL)                                    -->
-  <!-- TODO: Measure exact mount position on real vehicle           -->
+  <!-- Camera: ZED X Back (GMSL) — optional, off by default         -->
+  <!-- Serial 49910017 repurposed to zed_front; frame retained for  -->
+  <!-- documentation. Enable via: xacro ... enable_zed_back:=true   -->
   <!-- ============================================================ -->
-  <link name="zed_back_camera_center">
-    <visual>
-      <geometry>
-        <box size="0.04 0.17 0.03"/>
-      </geometry>
-      <material name="dark_grey"/>
-    </visual>
-  </link>
-  <joint name="zed_back_joint" type="fixed">
-    <parent link="base_link"/>
-    <child link="zed_back_camera_center"/>
-    <!-- TODO: Measure on vehicle. Approximate: rear center, facing back -->
-    <origin xyz="-0.75 0.0 0.6" rpy="0 0 3.14159"/>
-  </joint>
+  <xacro:if value="$(arg enable_zed_back)">
+    <link name="zed_back_camera_center">
+      <visual>
+        <geometry>
+          <box size="0.04 0.17 0.03"/>
+        </geometry>
+        <material name="dark_grey"/>
+      </visual>
+    </link>
+    <joint name="zed_back_joint" type="fixed">
+      <parent link="base_link"/>
+      <child link="zed_back_camera_center"/>
+      <!-- TODO: Measure on vehicle. Approximate: rear center, facing back -->
+      <origin xyz="-0.75 0.0 0.6" rpy="0 0 3.14159"/>
+    </joint>
+  </xacro:if>
 </robot>

Commit message: Live-tune HSV params + bake measured sensor mounts into URDF
- Declare 13 HSV pipeline params on perception_node with IntegerRange/
  FloatingPointRange descriptors so ros2 param set / rqt_reconfigure
  drive them. _on_set_params validates HSV bounds + low<=high atomically.
- HSVPipeline re-reads bounds, blur, adaptive_k, class IDs, and the ROI
  polygon from self.params on every run() so live tuning takes effect on
  the next frame.
- New test_hsv_live_tuning.py pins the contract end-to-end (5 tests,
  mutates params dict between successive run() calls).
- URDF: replace placeholder sensor mounts with measured offsets from
  the chassis sketch (origin = Xsens body, 0.5 m above ground).
  base_link sits at the IMU per the sketch convention; base_footprint
  joint drops -0.5 m to ground. RealSense link removed (unit not on
  robot).

Co-Authored-By: Claude Opus 4.7 (1M context) <noreply@anthropic.com>

File: src/avros_bringup/urdf/avros.urdf.xacro (robot description, xacro)
@@ -1,18 +1,24 @@
 <?xml version="1.0"?>
 <robot xmlns:xacro="http://www.ros.org/wiki/xacro" name="avros">
-  <!-- Vehicle parameters -->
-  <xacro:property name="wheelbase" value="1.23"/>
-  <xacro:property name="track_width" value="0.9"/>
+  <!-- Vehicle parameters (chassis box dimensions, not wheelbase) -->
+  <xacro:property name="chassis_length" value="1.23"/>
+  <xacro:property name="chassis_width"  value="0.9"/>
+  <xacro:property name="chassis_height" value="0.4"/>
   <!-- Optional frames. Pass via xacro args, e.g. xacro avros.urdf.xacro enable_zed_back:=true -->
   <xacro:arg name="enable_zed_back" default="false"/>
   <!-- ============================================================ -->
-  <!-- base_link: center of rear axle at ground level               -->
+  <!-- base_link: coincident with the Xsens body — that's the       -->
+  <!-- origin every sensor offset on the chassis was measured from. -->
+  <!-- Sits 0.5 m above ground at the chassis geometric center.     -->
+  <!-- The chassis box visual is shifted DOWN by Xsens height so it -->
+  <!-- still renders sitting on the floor in RViz/Foxglove.         -->
   <!-- ============================================================ -->
+  <xacro:property name="xsens_height" value="0.500"/>
   <link name="base_link">
     <visual>
       <geometry>
-        <box size="${wheelbase} ${track_width} 0.4"/>
+        <box size="${chassis_length} ${chassis_width} ${chassis_height}"/>
       </geometry>
-      <origin xyz="${wheelbase/2} 0 0.3" rpy="0 0 0"/>
+      <origin xyz="0 0 ${chassis_height/2 - xsens_height}" rpy="0 0 0"/>
       <material name="grey">
         <color rgba="0.5 0.5 0.5 0.8"/>
@@ -21,7 +27,7 @@
     <collision>
       <geometry>
-        <box size="${wheelbase} ${track_width} 0.4"/>
+        <box size="${chassis_length} ${chassis_width} ${chassis_height}"/>
       </geometry>
-      <origin xyz="${wheelbase/2} 0 0.3" rpy="0 0 0"/>
+      <origin xyz="0 0 ${chassis_height/2 - xsens_height}" rpy="0 0 0"/>
     </collision>
     <inertial>
@@ -37,5 +43,6 @@
     <parent link="base_link"/>
     <child link="base_footprint"/>
-    <origin xyz="0 0 0" rpy="0 0 0"/>
+    <!-- Drop straight down by xsens_height so base_footprint sits on the floor. -->
+    <origin xyz="0 0 ${-xsens_height}" rpy="0 0 0"/>
   </joint>
   <!-- ============================================================ -->
@@ -56,6 +63,6 @@
     <parent link="base_link"/>
     <child link="imu_link"/>
-    <!-- TODO: Measure on vehicle. Approximate: centered, roof height -->
-    <origin xyz="0.6 0.0 0.8" rpy="0 0 0"/>
+    <!-- Xsens body IS base_link (sketch convention). Zero offset. -->
+    <origin xyz="0 0 0" rpy="0 0 0"/>
   </joint>
   <!-- ============================================================ -->
@@ -76,26 +83,6 @@
     <parent link="base_link"/>
     <child link="velodyne"/>
-    <!-- TODO: Measure on vehicle. Approximate: centered, above roof -->
-    <origin xyz="0.6 0.0 1.0" rpy="0 0 0"/>
-  </joint>
-  <!-- ============================================================ -->
-  <!-- Camera: Intel RealSense D435i                                -->
-  <!-- TODO: Measure exact mount position on real vehicle           -->
-  <!-- ============================================================ -->
-  <link name="camera_link">
-    <visual>
-      <geometry>
-        <box size="0.025 0.09 0.025"/>
-      </geometry>
-      <material name="silver">
-        <color rgba="0.75 0.75 0.75 1"/>
-      </material>
-    </visual>
-  </link>
-  <joint name="camera_joint" type="fixed">
-    <parent link="base_link"/>
-    <child link="camera_link"/>
-    <!-- TODO: Measure on vehicle. Approximate: front, roof height -->
-    <origin xyz="1.0 0.0 0.8" rpy="0 0 0"/>
+    <!-- Sketch 2026-04-25: 3.5" forward, 6.25" up from Xsens, centerline. -->
+    <origin xyz="0.089 0.0 0.159" rpy="0 0 0"/>
   </joint>
   <!-- ============================================================ -->
@@ -114,6 +101,7 @@
     <parent link="base_link"/>
     <child link="zed_front_camera_link"/>
-    <!-- TODO: Measure on vehicle. Approximate: front center, roof height, facing +X -->
-    <origin xyz="1.0 0.0 0.9" rpy="0 0 0"/>
+    <!-- Sketch 2026-04-25: 15.625" forward, 2.25" above Xsens, centerline.
+         Faces +X (forward). -->
+    <origin xyz="0.397 0.0 0.057" rpy="0 0 0"/>
   </joint>
   <!-- ============================================================ -->
@@ -121,17 +109,14 @@
   <!-- TODO: Measure exact mount position on real vehicle           -->
   <!-- ============================================================ -->
-  <link name="zed_left_camera_center">
-    <visual>
-      <geometry>
-        <box size="0.04 0.17 0.03"/>
-      </geometry>
-      <material name="dark_grey"/>
-    </visual>
-  </link>
-  <joint name="zed_left_joint" type="fixed">
+  <xacro:zed_camera name="zed_left" model="zedx">
+    <origin xyz="0 0 0" rpy="0 0 0"/>
+  </xacro:zed_camera>
+  <joint name="zed_left_mount_joint" type="fixed">
     <parent link="base_link"/>
-    <child link="zed_left_camera_center"/>
-    <!-- TODO: Measure on vehicle. Approximate: left side, facing left -->
-    <origin xyz="-0.6 0.35 0.6" rpy="0 0 1.5708"/>
+    <child link="zed_left_camera_link"/>
+    <!-- Sketch 2026-04-25: 3.875" forward, 11.25" left of centerline,
+         2.25" above Xsens. Faces +Y (left). Sketch convention had
+         left=negative; flipped to ROS REP-103 (left=positive). -->
+    <origin xyz="0.098 0.286 0.057" rpy="0 0 1.5708"/>
   </joint>
   <!-- ============================================================ -->
@@ -139,17 +124,13 @@
   <!-- TODO: Measure exact mount position on real vehicle           -->
   <!-- ============================================================ -->
-  <link name="zed_right_camera_center">
-    <visual>
-      <geometry>
-        <box size="0.04 0.17 0.03"/>
-      </geometry>
-      <material name="dark_grey"/>
-    </visual>
-  </link>
-  <joint name="zed_right_joint" type="fixed">
+  <xacro:zed_camera name="zed_right" model="zedx">
+    <origin xyz="0 0 0" rpy="0 0 0"/>
+  </xacro:zed_camera>
+  <joint name="zed_right_mount_joint" type="fixed">
     <parent link="base_link"/>
-    <child link="zed_right_camera_center"/>
-    <!-- TODO: Measure on vehicle. Approximate: right side, facing right -->
-    <origin xyz="0.6 0.35 0.6" rpy="0 0 -1.5708"/>
+    <child link="zed_right_camera_link"/>
+    <!-- Sketch 2026-04-25: 3.875" forward, 11.25" right of centerline,
+         2.25" above Xsens. Faces -Y (right). -->
+    <origin xyz="0.098 -0.286 0.057" rpy="0 0 -1.5708"/>
   </joint>
   <!-- ============================================================ -->

Commit message: Move base_link back to ground level (standard convention)
Switching from convention "b" (base_link at IMU) back to convention "a"
(base_link at chassis center, ground level). Same physical sensor
positions, just bake the IMU's 0.5 m mounting height into each
sensor's Z offset instead of carrying it via base_footprint.

Why: 95% of public ROS2 / Nav2 code assumes base_link at ground level.
The kiwicampus semantic_segmentation_layer was producing internal
tiles correctly but never propagating them into the master local_costmap
when base_link was elevated — the most likely silent breakage.

- base_link.visual / .collision: re-centered (origin xyz="0 0 0.2" instead
  of "0 0 -0.3") so the chassis box renders sitting on the floor.
- base_footprint joint: zero offset, coincident with base_link.
- imu_link: now (0, 0, 0.5).
- velodyne, zed_front, zed_left, zed_right: Z is now xsens_height (0.5)
  plus the per-sketch local offset.

Co-Authored-By: Claude Opus 4.7 (1M context) <noreply@anthropic.com>

File: src/avros_bringup/urdf/avros.urdf.xacro (robot description, xacro)
@@ -8,9 +8,9 @@
   <xacro:arg name="enable_zed_back" default="false"/>
   <!-- ============================================================ -->
-  <!-- base_link: coincident with the Xsens body — that's the       -->
-  <!-- origin every sensor offset on the chassis was measured from. -->
-  <!-- Sits 0.5 m above ground at the chassis geometric center.     -->
-  <!-- The chassis box visual is shifted DOWN by Xsens height so it -->
-  <!-- still renders sitting on the floor in RViz/Foxglove.         -->
+  <!-- base_link: chassis geometric center at ground level.          -->
+  <!-- Standard ROS / Nav2 convention so robot_radius inflates       -->
+  <!-- around the centroid and downstream tools (Nav2, AMCL,         -->
+  <!-- robot_localization) work without surprise. Sensor offsets     -->
+  <!-- below have the IMU's 0.5 m mounting height baked into Z.      -->
   <!-- ============================================================ -->
   <xacro:property name="xsens_height" value="0.500"/>
@@ -20,5 +20,5 @@
         <box size="${chassis_length} ${chassis_width} ${chassis_height}"/>
       </geometry>
-      <origin xyz="0 0 ${chassis_height/2 - xsens_height}" rpy="0 0 0"/>
+      <origin xyz="0 0 ${chassis_height/2}" rpy="0 0 0"/>
       <material name="grey">
         <color rgba="0.5 0.5 0.5 0.8"/>
@@ -29,5 +29,5 @@
         <box size="${chassis_length} ${chassis_width} ${chassis_height}"/>
       </geometry>
-      <origin xyz="0 0 ${chassis_height/2 - xsens_height}" rpy="0 0 0"/>
+      <origin xyz="0 0 ${chassis_height/2}" rpy="0 0 0"/>
     </collision>
     <inertial>
@@ -37,5 +37,5 @@
   </link>
   <!-- ============================================================ -->
-  <!-- base_footprint: ground projection of base_link               -->
+  <!-- base_footprint: coincident with base_link (already on ground) -->
   <!-- ============================================================ -->
   <link name="base_footprint"/>
@@ -43,6 +43,5 @@
     <parent link="base_link"/>
     <child link="base_footprint"/>
-    <!-- Drop straight down by xsens_height so base_footprint sits on the floor. -->
-    <origin xyz="0 0 ${-xsens_height}" rpy="0 0 0"/>
+    <origin xyz="0 0 0" rpy="0 0 0"/>
   </joint>
   <!-- ============================================================ -->
@@ -63,6 +62,6 @@
     <parent link="base_link"/>
     <child link="imu_link"/>
-    <!-- Xsens body IS base_link (sketch convention). Zero offset. -->
-    <origin xyz="0 0 0" rpy="0 0 0"/>
+    <!-- Sketch 2026-04-25: Xsens at chassis center, 0.5 m above ground. -->
+    <origin xyz="0 0 ${xsens_height}" rpy="0 0 0"/>
   </joint>
   <!-- ============================================================ -->
@@ -83,6 +82,7 @@
     <parent link="base_link"/>
     <child link="velodyne"/>
-    <!-- Sketch 2026-04-25: 3.5" forward, 6.25" up from Xsens, centerline. -->
-    <origin xyz="0.089 0.0 0.159" rpy="0 0 0"/>
+    <!-- Sketch 2026-04-25: 3.5" forward, 6.25" up from Xsens.
+         Xsens is xsens_height above base_link, so Z = xsens_height + 0.159. -->
+    <origin xyz="0.089 0.0 ${xsens_height + 0.159}" rpy="0 0 0"/>
   </joint>
   <!-- ============================================================ -->
@@ -101,7 +101,7 @@
     <parent link="base_link"/>
     <child link="zed_front_camera_link"/>
-    <!-- Sketch 2026-04-25: 15.625" forward, 2.25" above Xsens, centerline.
-         Faces +X (forward). -->
-    <origin xyz="0.397 0.0 0.057" rpy="0 0 0"/>
+    <!-- Sketch 2026-04-25: 15.625" forward, 2.25" above Xsens.
+         Z = xsens_height + 0.057. Faces +X (forward). -->
+    <origin xyz="0.397 0.0 ${xsens_height + 0.057}" rpy="0 0 0"/>
   </joint>
   <!-- ============================================================ -->
@@ -116,7 +116,7 @@
     <child link="zed_left_camera_link"/>
     <!-- Sketch 2026-04-25: 3.875" forward, 11.25" left of centerline,
-         2.25" above Xsens. Faces +Y (left). Sketch convention had
-         left=negative; flipped to ROS REP-103 (left=positive). -->
-    <origin xyz="0.098 0.286 0.057" rpy="0 0 1.5708"/>
+         2.25" above Xsens. Z = xsens_height + 0.057. Faces +Y (left).
+         Sketch convention had left=negative; flipped to ROS REP-103. -->
+    <origin xyz="0.098 0.286 ${xsens_height + 0.057}" rpy="0 0 1.5708"/>
   </joint>
   <!-- ============================================================ -->
@@ -131,6 +131,6 @@
     <child link="zed_right_camera_link"/>
     <!-- Sketch 2026-04-25: 3.875" forward, 11.25" right of centerline,
-         2.25" above Xsens. Faces -Y (right). -->
-    <origin xyz="0.098 -0.286 0.057" rpy="0 0 -1.5708"/>
+         2.25" above Xsens. Z = xsens_height + 0.057. Faces -Y (right). -->
+    <origin xyz="0.098 -0.286 ${xsens_height + 0.057}" rpy="0 0 -1.5708"/>
   </joint>
   <!-- ============================================================ -->
