Commit message: urdf: resurvey chassis geometry from cpp_avl_igvc, fix ZED front mount
Adopts the cleaner chassis model from cpp_avl_igvc/igvc_description
(2026-05-06 resurvey of the same physical AVL IGVC chassis): replaces
the single 1.23 x 0.9 x 0.4 m box with a four-piece model — main
chassis box (0.743 x 0.6795 x 0.3747), top sensor platform (0.5842
x 0.5715 x 0.1461), and left/right tread enclosures (0.8255 x 0.0889
x 0.1397 each, centered ±0.3653 m off the centerline).

  - IMU anchor (xsens_height): 0.500 → 0.5556 m (21.875 in surveyed)
  - All component positions expressed relative to the IMU.

ZED front mount corrected from sketch estimate to surveyed value:
  - was: 0.397 m fwd, +0.057 m above IMU (15.625" fwd, 2.25" up)
  - now: 0.6795 m fwd, -0.108 m below IMU (26.75" fwd, 4.25" down)
  - prior estimate was off by ~28 cm in the forward direction.

Co-Authored-By: Claude Opus 4.7 (1M context) <noreply@anthropic.com>

File: src/avros_bringup/urdf/avros.urdf.xacro (robot description, xacro)
@@ -1,8 +1,4 @@
 <?xml version="1.0"?>
 <robot xmlns:xacro="http://www.ros.org/wiki/xacro" name="avros">
-  <!-- Vehicle parameters (chassis box dimensions, not wheelbase) -->
-  <xacro:property name="chassis_length" value="1.23"/>
-  <xacro:property name="chassis_width"  value="0.9"/>
-  <xacro:property name="chassis_height" value="0.4"/>
   <!-- Optional frames. Pass via xacro args, e.g. xacro avros.urdf.xacro enable_zed_back:=true -->
   <xacro:arg name="enable_zed_back" default="false"/>
@@ -12,22 +8,84 @@
   <!-- around the centroid and downstream tools (Nav2, AMCL,         -->
   <!-- robot_localization) work without surprise. Sensor offsets     -->
-  <!-- below have the IMU's 0.5 m mounting height baked into Z.      -->
-  <!-- ============================================================ -->
-  <xacro:property name="xsens_height" value="0.500"/>
+  <!-- below have the IMU mounting height baked into Z via the       -->
+  <!-- xsens_height anchor.                                          -->
+  <!--                                                               -->
+  <!-- Chassis geometry adopted from cpp_avl_igvc/igvc_description   -->
+  <!-- (calebhylkema, 2026-05-06). Their team re-surveyed the same   -->
+  <!-- physical AVL IGVC chassis with cleaner two-box + tread        -->
+  <!-- enclosures instead of our prior single 1.23×0.9×0.4 box.      -->
+  <!-- All component positions are expressed relative to the IMU at  -->
+  <!-- xsens_height above ground.                                    -->
+  <!-- ============================================================ -->
+  <xacro:property name="xsens_height" value="0.5556"/>  <!-- 21.875 in -->
+  <!-- Main chassis box: 29.25 × 26.75 × 14.75 in -->
+  <xacro:property name="main_length" value="0.7430"/>
+  <xacro:property name="main_width"  value="0.6795"/>
+  <xacro:property name="main_height" value="0.3747"/>
+  <!-- Top sensor platform: 23.00 × 22.50 × 5.75 in -->
+  <xacro:property name="top_length" value="0.5842"/>
+  <xacro:property name="top_width"  value="0.5715"/>
+  <xacro:property name="top_height" value="0.1461"/>
+  <!-- Tread enclosures: 32.5 × 3.5 × 5.5 in, centered ±0.3653 m off centerline -->
+  <xacro:property name="tread_length" value="0.8255"/>
+  <xacro:property name="tread_width"  value="0.0889"/>
+  <xacro:property name="tread_height" value="0.1397"/>
+  <xacro:property name="tread_y"      value="0.3653"/>
   <link name="base_link">
-    <visual>
-      <geometry>
-        <box size="${chassis_length} ${chassis_width} ${chassis_height}"/>
-      </geometry>
-      <origin xyz="0 0 ${chassis_height/2}" rpy="0 0 0"/>
-      <material name="grey">
-        <color rgba="0.5 0.5 0.5 0.8"/>
-      </material>
-    </visual>
-    <collision>
-      <geometry>
-        <box size="${chassis_length} ${chassis_width} ${chassis_height}"/>
-      </geometry>
-      <origin xyz="0 0 ${chassis_height/2}" rpy="0 0 0"/>
+    <!-- Main chassis box -->
+    <visual>
+      <origin xyz="0.3143 0 ${xsens_height - 0.2191}" rpy="0 0 0"/>
+      <geometry>
+        <box size="${main_length} ${main_width} ${main_height}"/>
+      </geometry>
+      <material name="grey"><color rgba="0.55 0.55 0.55 0.8"/></material>
+    </visual>
+    <collision>
+      <origin xyz="0.3143 0 ${xsens_height - 0.2191}" rpy="0 0 0"/>
+      <geometry>
+        <box size="${main_length} ${main_width} ${main_height}"/>
+      </geometry>
+    </collision>
+    <!-- Top sensor platform -->
+    <visual>
+      <origin xyz="0.1143 0 ${xsens_height + 0.0413}" rpy="0 0 0"/>
+      <geometry>
+        <box size="${top_length} ${top_width} ${top_height}"/>
+      </geometry>
+      <material name="light_grey"><color rgba="0.70 0.70 0.70 0.8"/></material>
+    </visual>
+    <collision>
+      <origin xyz="0.1143 0 ${xsens_height + 0.0413}" rpy="0 0 0"/>
+      <geometry>
+        <box size="${top_length} ${top_width} ${top_height}"/>
+      </geometry>
+    </collision>
+    <!-- Left tread enclosure -->
+    <visual>
+      <origin xyz="0.3143 ${tread_y} ${xsens_height - 0.4763}" rpy="0 0 0"/>
+      <geometry>
+        <box size="${tread_length} ${tread_width} ${tread_height}"/>
+      </geometry>
+      <material name="dark_grey"><color rgba="0.25 0.25 0.25 0.9"/></material>
+    </visual>
+    <collision>
+      <origin xyz="0.3143 ${tread_y} ${xsens_height - 0.4763}" rpy="0 0 0"/>
+      <geometry>
+        <box size="${tread_length} ${tread_width} ${tread_height}"/>
+      </geometry>
+    </collision>
+    <!-- Right tread enclosure -->
+    <visual>
+      <origin xyz="0.3143 ${-tread_y} ${xsens_height - 0.4763}" rpy="0 0 0"/>
+      <geometry>
+        <box size="${tread_length} ${tread_width} ${tread_height}"/>
+      </geometry>
+      <material name="dark_grey"/>
+    </visual>
+    <collision>
+      <origin xyz="0.3143 ${-tread_y} ${xsens_height - 0.4763}" rpy="0 0 0"/>
+      <geometry>
+        <box size="${tread_length} ${tread_width} ${tread_height}"/>
+      </geometry>
     </collision>
     <inertial>
@@ -101,7 +159,9 @@
     <parent link="base_link"/>
     <child link="zed_front_camera_link"/>
-    <!-- Sketch 2026-04-25: 15.625" forward, 2.25" above Xsens.
-         Z = xsens_height + 0.057. Faces +X (forward). -->
-    <origin xyz="0.397 0.0 ${xsens_height + 0.057}" rpy="0 0 0"/>
+    <!-- Resurvey 2026-05-06 (cpp_avl_igvc): 26.75" forward, 4.25" below
+         IMU. Z = xsens_height - 0.108. Faces +X (forward). Replaces
+         prior estimate (15.625" forward, 2.25" above) which was off
+         by ~28 cm forward. -->
+    <origin xyz="0.6795 0.0 ${xsens_height - 0.108}" rpy="0 0 0"/>
   </joint>
   <!-- ============================================================ -->

Commit message: urdf: ZED front camera 15° downward pitch on mount bracket
Physical change to the robot — the ZED front camera was tilted 15°
downward on its bracket to keep the painted lane in frame at near
range. Previously the camera pointed level forward (rpy="0 0 0"),
so the lower portion of the field-of-view started at the horizon
and the near-field grass (closest 2-3m) was below the frame edge.
With 15° pitch down, the bottom of the FOV reaches ~0.5-1m in
front of the bumper at typical mounting height — much better
coverage of the lane right in front of the robot for the kiwicampus
semantic_segmentation_layer to project into the local costmap.

URDF semantics:
  pitch = +0.2618 rad (= +15°) rotates the camera-link frame's
  +X-forward axis toward -Z-down (right-hand rule on +Y),
  i.e. the camera ends up "looking at the ground" by 15°.

No other changes required:
  - perception_node uses TF chain base_link -> zed_front_camera_link
    -> zed_front_left_camera_frame_optical, so projection of mask
    pixels into the local costmap automatically incorporates the
    new orientation.
  - kiwicampus semantic_segmentation_layer queries TF at the cloud's
    timestamp — picks up the new transform on next launch.
  - costmap config (inflation_radius=0.65, etc.) is unchanged.

Must restart robot_state_publisher (i.e. the full launch tree) for
the new TF to take effect — runtime URDF reload is not supported.

Co-Authored-By: Claude Opus 4.7 (1M context) <noreply@anthropic.com>

File: src/avros_bringup/urdf/avros.urdf.xacro (robot description, xacro)
@@ -162,6 +162,9 @@
          IMU. Z = xsens_height - 0.108. Faces +X (forward). Replaces
          prior estimate (15.625" forward, 2.25" above) which was off
-         by ~28 cm forward. -->
-    <origin xyz="0.6795 0.0 ${xsens_height - 0.108}" rpy="0 0 0"/>
+         by ~28 cm forward.
+         2026-05-12: physically tilted 15° down on the bracket to keep
+         the lane in frame at near-range. pitch = +0.2618 rad rotates
+         the camera's +X-forward axis toward -Z-down. -->
+    <origin xyz="0.6795 0.0 ${xsens_height - 0.108}" rpy="0 ${radians(15)} 0"/>
   </joint>
   <!-- ============================================================ -->
